Commit message: Integrated D435 camera model

File: robots/panda_arm_hand.urdf.xacro (robot description, xacro)
@@ -18,5 +18,5 @@
     <xacro:include filename="$(find franka_panda_description)/robots/panda.transmission.xacro"/>
     <xacro:panda_arm in_gazebo="true" />
-    <xacro:panda_gazebo robot_name="$(arg robot_name)" load_gripper="$(arg load_gripper)"/>
+    <xacro:panda_gazebo       robot_name="$(arg robot_name)" load_gripper="$(arg load_gripper)"/>
     <xacro:panda_transmission robot_name="$(arg robot_name)" load_gripper="$(arg load_gripper)"/>
   </xacro:if>
@@ -26,10 +26,6 @@
   <!-- Intel Realsense Camera -->
   <xacro:if value="$(arg intel_realsense)">
-    <xacro:include filename="${urdf_path}/camera/_d435.urdf.xacro"/>
-    <joint name="intel_realsense_joint" type="fixed">
-      <origin xyz="0 -0.4 0.6" rpy="0 0.4 ${pi + -0.5}"/>
-      <parent link="$(arg robot_name)_base_link"/>
-      <child link="intel_realsense_bottom_screw_frame"/>
-    </joint>
+    <xacro:include filename="$(find franka_panda_description)/urdf/camera/_d435.urdf.xacro" />
+    <xacro:sensor_d435 parent="panda_link0" xyz="1.5 0 0.6" rpy="0 0.3 ${pi}"/>
   </xacro:if>
 </robot>

File: urdf/camera/_d435.gazebo.xacro (robot description, xacro)
@@ -6,5 +6,5 @@
 -->
 <robot xmlns:xacro="http://ros.org/wiki/xacro">
-  <xacro:macro name="intel_camera_link" params="camera_name reference_link topics_ns depth_optical_frame color_optical_frame infrared1_optical_frame infrared2_optical_frame" >
+  <xacro:macro name="gazebo_d435" params="camera_name reference_link topics_ns depth_optical_frame color_optical_frame infrared1_optical_frame infrared2_optical_frame" >
     <!-- Load parameters to model's main link-->
     <xacro:property name="deg_to_rad" value="0.01745329251994329577" />

File: urdf/camera/_d435.urdf.xacro (robot description, xacro)
@@ -6,8 +6,8 @@
 aluminum peripherial evaluation case.
 -->
-<robot name="intel_realsense" xmlns:xacro="http://ros.org/wiki/xacro">
+<robot name="sensor_d435" xmlns:xacro="http://ros.org/wiki/xacro">
   <!--File includes-->
   <xacro:include filename="$(find franka_panda_description)/urdf/camera/_d435.gazebo.xacro"/>
-  <xacro:macro name="sensor_d435" params="name:=camera topics_ns:=camera parent *origin">
+  <xacro:macro name="sensor_d435" params="name:=camera topics_ns:=camera parent xyz rpy">
     <xacro:property name="M_PI" value="3.1415926535897931" />
     <!-- The following values are approximate, and the camera node
@@ -32,9 +32,9 @@
     </material>
     <!-- camera body, with origin at bottom screw mount -->
-    <!--<joint name="${name}_joint" type="fixed">
-      <xacro:insert_block name="origin" />
+    <joint name="${name}_joint" type="fixed">
       <parent link="${parent}"/>
       <child link="${name}_bottom_screw_frame" />
-    </joint> -->
+      <origin xyz="${xyz}" rpy="${rpy}"/>
+    </joint>
     <link name="${name}_bottom_screw_frame"/>
     <joint name="${name}_link_joint" type="fixed">
@@ -43,10 +43,10 @@
       <child link="${name}_link" />
     </joint>
-    <link name="${name}_realsense_link">
+    <link name="${name}_link">
       <visual>
       <origin xyz="${d435_cam_mount_from_center_offset} ${-d435_cam_depth_py} 0" rpy="${M_PI/2} 0 ${M_PI/2}"/>
         <geometry>
           <!-- <box size="${d435_cam_width} ${d435_cam_height} ${d435_cam_depth}"/> -->
-          <mesh filename="package://realsense2_description/meshes/d435.dae" />
+          <mesh filename="package://franka_panda_description/meshes/camera/d435.dae" />
           <!--<mesh filename="package://realsense2_description/meshes/d435/d435.dae" />-->
         </geometry>

Commit message: Changed robot name

File: robots/panda_arm_hand.urdf.xacro (robot description, xacro)
@@ -3,11 +3,7 @@
   <xacro:arg name="robot_name"      default="panda"/>
   <xacro:arg name="load_gripper"    default="false"/>
-  <xacro:arg name="load_hand"       default="false" />
+  <xacro:arg name="load_hand"       default="true" />
   <xacro:arg name="load_gazebo"     default="false"/>
   <xacro:arg name="intel_realsense" default="true" />
-  <!-- ========================================================================================== -->
-  <!-- Set xacro properties -->
-  <xacro:property name="urdf_path"    value="$(find franka_panda_description)/urdf"/>
-  <!-- ========================================================================================== -->
   <!-- Panda Arm -->
   <xacro:include filename="$(find franka_panda_description)/robots/panda_arm.xacro"/>
