Commit message: noetic-devel

File: robots/panda.gazebo.xacro (robot description, xacro)
@@ -1,4 +1,11 @@
 <?xml version="1.0"?>
 <robot xmlns:xacro="http://www.ros.org/wiki/xacro">
+<!-- ROS control plugin -->
+    <gazebo>
+      <plugin name="gazebo_ros_control" filename="libgazebo_ros_control.so">
+        <!-- This tag gets rid of an error that popped up in version 8.6 -->
+        <legacyModeNS>true</legacyModeNS>
+      </plugin>
+    </gazebo>
     <xacro:macro name="panda_gazebo" params="robot_name load_gripper">
       <gazebo reference="${robot_name}_joint7">

File: robots/panda_arm.xacro (robot description, xacro)
@@ -2,4 +2,5 @@
 <robot xmlns:xacro="http://www.ros.org/wiki/xacro" name="panda">
   <xacro:macro name="panda_arm" params="arm_id:='panda' description_pkg:='franka_panda_description' connected_to:='' in_gazebo='false' xyz:='0 0 0' rpy:='0 0 0'">
+    <xacro:property name="joint_damping" value="1.0"/>
     <!-- If using custom frame with ${connected_to} param, make sure 'world' frame exists in its TF tree -->
     <xacro:if value="${connected_to == ''}">
@@ -24,9 +25,10 @@
         </geometry>
       </visual>
-      <collision>
+      <!--<collision>
         <geometry>
           <mesh filename="package://${description_pkg}/meshes/collision/link0.stl"/>
         </geometry>
       </collision>
+      -->
       <xacro:unless value="${in_gazebo == 'false'}">
         <inertial>
@@ -43,9 +45,10 @@
         </geometry>
       </visual>
-      <collision>
+      <!--<collision>
         <geometry>
           <mesh filename="package://${description_pkg}/meshes/collision/link1.stl"/>
         </geometry>
       </collision>
+      -->
       <inertial>
         <origin xyz="3.875e-03 2.081e-03 -0.1750" rpy="0 0 0"/>
@@ -69,9 +72,10 @@
         </geometry>
       </visual>
-      <collision>
+      <!--<collision>
         <geometry>
           <mesh filename="package://${description_pkg}/meshes/collision/link2.stl"/>
         </geometry>
       </collision>
+      -->
       <inertial>
         <origin xyz="-3.141e-03 -2.872e-02 3.495e-03" rpy="0 0 0"/>
@@ -95,9 +99,10 @@
         </geometry>
       </visual>
-      <collision>
+      <!--<collision>
         <geometry>
           <mesh filename="package://${description_pkg}/meshes/collision/link3.stl"/>
         </geometry>
       </collision>
+      -->
       <inertial>
         <origin xyz="2.7518e-02 3.9252e-02 -6.6502e-02" rpy="0 0 0"/>
@@ -121,4 +126,5 @@
         </geometry>
       </visual>
+      <!--
       <collision>
         <geometry>
@@ -126,4 +132,5 @@
         </geometry>
       </collision>
+      -->
       <inertial>
         <origin xyz="-5.317e-02 1.04419e-01 2.7454e-02" rpy="0 0 0"/>
@@ -147,9 +154,10 @@
         </geometry>
       </visual>
-      <collision>
+      <!--<collision>
         <geometry>
           <mesh filename="package://${description_pkg}/meshes/collision/link5.stl"/>
         </geometry>
       </collision>
+      -->
       <inertial>
         <origin xyz="-1.1953e-02 4.1065e-02 -3.8437e-02" rpy="0 0 0"/>
@@ -173,4 +181,5 @@
         </geometry>
       </visual>
+      <!--
       <collision>
         <geometry>
@@ -178,4 +187,5 @@
         </geometry>
       </collision>
+      -->
       <inertial>
         <origin xyz="6.0149e-02 -1.4117e-02 -1.0517e-02" rpy="0 0 0"/>
@@ -199,9 +209,10 @@
         </geometry>
       </visual>
-      <collision>
+      <!--<collision>
         <geometry>
           <mesh filename="package://${description_pkg}/meshes/collision/link7.stl"/>
         </geometry>
       </collision>
+      -->
       <inertial>
         <origin xyz="1.0517e-02 -4.252e-03 6.1597e-02" rpy="0 0 0"/>

File: robots/panda_arm_hand.urdf.xacro (robot description, xacro)
@@ -1,23 +1,38 @@
 <?xml version="1.0"?>
 <robot xmlns:xacro="http://www.ros.org/wiki/xacro" name="panda">
-  <xacro:arg name="robot_name" default="panda"/>
-  <xacro:arg name="load_gripper" default="true"/>
-  <xacro:arg name="load_gazebo" default="false"/>
+  <xacro:arg name="robot_name"      default="panda"/>
+  <xacro:arg name="load_gripper"    default="false"/>
+  <xacro:arg name="load_hand"       default="true" />
+  <xacro:arg name="realsense"       default="d435" />
   <xacro:arg name="use_gazebo_control" default="false"/>
   <xacro:arg name="connected_to" default=""/> <!-- If using a different frame with ${connected_to} param, make sure 'world' frame exists in the TF tree -->
+  <!-- Panda Arm -->
   <xacro:include filename="$(find franka_panda_description)/robots/panda_arm.xacro"/>
+  <!-- Gazebo -->
+  <xacro:include filename="$(find franka_panda_description)/robots/panda.gazebo.xacro"       />
+  <xacro:include filename="$(find franka_panda_description)/robots/panda.transmission.xacro" />
+  <xacro:panda_arm          arm_id="$(arg robot_name)" in_gazebo="true" xyz="0 0 0" rpy="0 0 0" />
+  <xacro:panda_gazebo       robot_name="$(arg robot_name)" load_gripper="$(arg load_gripper)"/>
+  <xacro:panda_transmission robot_name="$(arg robot_name)" load_gripper="$(arg load_gripper)"/>
+  <!-- Default Panda Gripper -->
   <xacro:if value="$(arg load_gripper)">
     <xacro:include filename="$(find franka_panda_description)/robots/hand.xacro"/>
-    <xacro:hand ns="panda" rpy="0 0 ${-pi/4}" connected_to="panda_link8"/>
+    <xacro:hand ns="panda" rpy="0 0 ${pi/4}" connected_to="panda_link8"/>
   </xacro:if>
-  <xacro:if value="$(arg load_gazebo)">
-    <xacro:include filename="$(find franka_panda_description)/robots/panda.gazebo.xacro"/>
-    <xacro:include filename="$(find franka_panda_description)/robots/panda.transmission.xacro"/>
-    <xacro:panda_arm in_gazebo="true"  connected_to="$(arg connected_to)"/>
-    <xacro:panda_gazebo robot_name="$(arg robot_name)" load_gripper="$(arg load_gripper)"/>
-    <xacro:panda_transmission robot_name="$(arg robot_name)" load_gripper="$(arg load_gripper)" use_gazebo_control="$(arg use_gazebo_control)"/>
+  <!-- Hithand, joint between hithand_base and panda_link_8 inside hithand.xacro-->
+  <xacro:if value="$(arg load_hand)">
+    <xacro:include filename="$(find hithand_description)/urdf/hithand.xacro"/>
+    <xacro:hithand attached="true" ns="panda" rpy="0 0 0" parent="panda_link8"/>
   </xacro:if>
-  <xacro:unless value="$(arg load_gazebo)">
-    <xacro:panda_arm />
-  </xacro:unless>
+  <!-- Intel Realsense D435 Camera -->
+  <xacro:if value="$(eval realsense == 'd435')">
+    <xacro:include filename="$(find franka_panda_description)/urdf/camera/_d435.urdf.xacro" />
+    <!-- <xacro:sensor_d435 parent="panda_link0" xyz="0.86 -1 0.35" rpy="0 0.3 ${pi/2}"/>  -->
+    <xacro:sensor_d435 parent="panda_link0" xyz="0.5 -0.75 0.35" rpy="0 0.3 ${pi/2}"/>
+  </xacro:if>
+  <!-- Intel Realsense D415 Camera -->
+  <xacro:if value="$(eval realsense == 'd415')">
+    <xacro:include filename="$(find franka_panda_description)/urdf/camera/_d415.urdf.xacro" />
+    <xacro:sensor_d415 parent="panda_link0" xyz="0.5 -0.85 0.35" rpy="0 0.3 ${pi/2}"/>
+  </xacro:if>
 </robot>
