Commit message: Added camera

File: robots/panda_arm.xacro (robot description, xacro)
@@ -1,5 +1,6 @@
 <?xml version='1.0'?>
 <robot xmlns:xacro="http://www.ros.org/wiki/xacro" name="panda">
-  <xacro:macro name="panda_arm" params="arm_id:='panda' description_pkg:='franka_description' connected_to:=''  in_gazebo='false' xyz:='0 0 0' rpy:='0 0 0'">
+  <xacro:macro name="panda_arm" params="arm_id:='panda' description_pkg:='franka_description'
+					connected_to:=''  in_gazebo='false' xyz:='0 0 0' rpy:='0 0 0'">
     <xacro:unless value="${not connected_to}">
       <joint name="${arm_id}_joint_${connected_to}" type="fixed">

File: robots/panda_arm_hand.urdf.xacro (robot description, xacro)
@@ -4,4 +4,9 @@
   <xacro:arg name="load_gripper" default="true"/>
   <xacro:arg name="load_gazebo" default="false"/>
+  <xacro:arg name="intel_realsense" default="true"/>
+  <!-- ========================================================================================== -->
+  <!-- Set xacro properties -->
+  <xacro:property name="urdf_path"    value="$(find franka_panda_description)/urdf"/>
+  <!-- ========================================================================================== -->
   <xacro:include filename="$(find franka_panda_description)/robots/panda_arm.xacro"/>
   <xacro:if value="$(arg load_gripper)">
@@ -19,3 +24,12 @@
     <xacro:panda_arm />
   </xacro:unless>
+  <!-- Intel Realsense Camera -->
+  <xacro:if value="$(arg intel_realsense)">
+    <xacro:include filename="${urdf_path}/camera/_d435.urdf.xacro"/>
+    <joint name="intel_realsense_joint" type="fixed">
+      <origin xyz="0 -0.4 0.6" rpy="0 0.4 ${pi + -0.5}"/>
+      <parent link="$(arg robot_name)_base_link"/>
+      <child link="intel_realsense_bottom_screw_frame"/>
+    </joint>
+  </xacro:if>
 </robot>

Commit message: Added hithand, displays correctly in simulation, fails to control

File: robots/panda_arm.xacro (robot description, xacro)
@@ -2,5 +2,6 @@
 <robot xmlns:xacro="http://www.ros.org/wiki/xacro" name="panda">
   <xacro:macro name="panda_arm" params="arm_id:='panda' description_pkg:='franka_description'
-					connected_to:=''  in_gazebo='false' xyz:='0 0 0' rpy:='0 0 0'">
+				connected_to:='' in_gazebo='false' xyz:='0 0 0' rpy:='0 0 0'">
+    <xacro:property name="joint_damping" value="1.0"/>
     <xacro:unless value="${not connected_to}">
       <joint name="${arm_id}_joint_${connected_to}" type="fixed">
@@ -10,5 +11,4 @@
       </joint>
     </xacro:unless>
-    <xacro:property name="joint_damping" value="1.0"/>
     <xacro:unless value="${in_gazebo == 'false'}">
       <link name="world" />

File: robots/panda_arm_hand.urdf.xacro (robot description, xacro)
@@ -1,21 +1,20 @@
 <?xml version="1.0"?>
 <robot xmlns:xacro="http://www.ros.org/wiki/xacro" name="panda">
-  <xacro:arg name="robot_name" default="panda"/>
-  <xacro:arg name="load_gripper" default="true"/>
-  <xacro:arg name="load_gazebo" default="false"/>
-  <xacro:arg name="intel_realsense" default="true"/>
+  <xacro:arg name="robot_name"      default="panda"/>
+  <xacro:arg name="load_gripper"    default="false"/>
+  <xacro:arg name="load_hand"       default="false" />
+  <xacro:arg name="load_gazebo"     default="false"/>
+  <xacro:arg name="intel_realsense" default="true" />
   <!-- ========================================================================================== -->
   <!-- Set xacro properties -->
   <xacro:property name="urdf_path"    value="$(find franka_panda_description)/urdf"/>
   <!-- ========================================================================================== -->
+  <!-- Panda Arm -->
   <xacro:include filename="$(find franka_panda_description)/robots/panda_arm.xacro"/>
-  <xacro:if value="$(arg load_gripper)">
-    <xacro:include filename="$(find franka_panda_description)/robots/hand.xacro"/>
-    <xacro:hand ns="panda" rpy="0 0 ${-pi/4}" connected_to="panda_link8"/>
-  </xacro:if>
+  <!-- Gazebo -->
   <xacro:if value="$(arg load_gazebo)">
-    <xacro:include filename="$(find franka_panda_description)/robots/panda.gazebo.xacro"/>
-    <xacro:include filename="$(find franka_panda_description)/robots/panda.transmission.xacro"/>
-    <xacro:panda_arm in_gazebo="true" />
+    <xacro:include filename="$(find franka_panda_description)/robots/panda.gazebo.xacro"       />
+    <xacro:include filename="$(find franka_panda_description)/robots/panda.transmission.xacro" />
+    <xacro:panda_arm in_gazebo="true" xyz="0 0 0" rpy="0 0 0" />
     <xacro:panda_gazebo       robot_name="$(arg robot_name)" load_gripper="$(arg load_gripper)"/>
     <xacro:panda_transmission robot_name="$(arg robot_name)" load_gripper="$(arg load_gripper)"/>
@@ -24,4 +23,14 @@
     <xacro:panda_arm />
   </xacro:unless>
+  <!-- Default Panda Gripper -->
+  <xacro:if value="$(arg load_gripper)">
+    <xacro:include filename="$(find franka_panda_description)/robots/hand.xacro"/>
+    <xacro:hand ns="panda" rpy="0 0 ${-pi/4}" connected_to="panda_link8"        />
+  </xacro:if>
+  <!-- Hithand -->
+  <xacro:if value="$(arg load_hand)">
+    <xacro:include filename="$(find hithand_description)/urdf/hithand.xacro"/>
+    <xacro:hithand attached="true" ns="panda" rpy="0 0 ${-pi/2}" parent="panda_link8"/>
+  </xacro:if>
   <!-- Intel Realsense Camera -->
   <xacro:if value="$(arg intel_realsense)">

Commit message: chore: remove unneccessary variables

File: robots/panda_arm.xacro (robot description, xacro)
@@ -1,5 +1,5 @@
 <?xml version='1.0'?>
 <robot xmlns:xacro="http://www.ros.org/wiki/xacro" name="panda">
-  <xacro:macro name="panda_arm" params="arm_id:='panda' description_pkg:='franka_description'
+  <xacro:macro name="panda_arm" params="arm_id:='panda' description_pkg:='franka_panda_description'
 				connected_to:='' in_gazebo='false' xyz:='0 0 0' rpy:='0 0 0'">
     <xacro:property name="joint_damping" value="1.0"/>
@@ -26,9 +26,9 @@
         </geometry>
       </visual>
-      <collision>
+      <!-- <collision>
         <geometry>
           <mesh filename="package://${description_pkg}/meshes/collision/link0.stl"/>
         </geometry>
-      </collision>
+      </collision> -->
       <xacro:unless value="${in_gazebo == 'false'}">
         <inertial>
@@ -45,9 +45,9 @@
         </geometry>
       </visual>
-      <collision>
+      <!-- <collision>
         <geometry>
           <mesh filename="package://${description_pkg}/meshes/collision/link1.stl"/>
         </geometry>
-      </collision>
+      </collision> -->
       <inertial>
         <origin xyz="3.875e-03 2.081e-03 -0.1750" rpy="0 0 0"/>
@@ -71,9 +71,9 @@
         </geometry>
       </visual>
-      <collision>
+      <!-- <collision>
         <geometry>
           <mesh filename="package://${description_pkg}/meshes/collision/link2.stl"/>
         </geometry>
-      </collision>
+      </collision> -->
       <inertial>
         <origin xyz="-3.141e-03 -2.872e-02 3.495e-03" rpy="0 0 0"/>
@@ -97,9 +97,9 @@
         </geometry>
       </visual>
-      <collision>
+      <!-- <collision>
         <geometry>
           <mesh filename="package://${description_pkg}/meshes/collision/link3.stl"/>
         </geometry>
-      </collision>
+      </collision> -->
       <inertial>
         <origin xyz="2.7518e-02 3.9252e-02 -6.6502e-02" rpy="0 0 0"/>
@@ -123,9 +123,9 @@
         </geometry>
       </visual>
-      <collision>
+      <!-- <collision>
         <geometry>
           <mesh filename="package://${description_pkg}/meshes/collision/link4.stl"/>
         </geometry>
-      </collision>
+      </collision> -->
       <inertial>
         <origin xyz="-5.317e-02 1.04419e-01 2.7454e-02" rpy="0 0 0"/>

File: robots/panda_arm_hand.urdf.xacro (robot description, xacro)
@@ -4,19 +4,13 @@
   <xacro:arg name="load_gripper"    default="false"/>
   <xacro:arg name="load_hand"       default="true" />
-  <xacro:arg name="load_gazebo"     default="false"/>
   <xacro:arg name="intel_realsense" default="true" />
   <!-- Panda Arm -->
   <xacro:include filename="$(find franka_panda_description)/robots/panda_arm.xacro"/>
   <!-- Gazebo -->
-  <xacro:if value="$(arg load_gazebo)">
-    <xacro:include filename="$(find franka_panda_description)/robots/panda.gazebo.xacro"       />
-    <xacro:include filename="$(find franka_panda_description)/robots/panda.transmission.xacro" />
-    <xacro:panda_arm          arm_id="$(arg robot_name)" in_gazebo="true" xyz="0 0 0" rpy="0 0 0" />
-    <xacro:panda_gazebo       robot_name="$(arg robot_name)" load_gripper="$(arg load_gripper)"/>
-    <xacro:panda_transmission robot_name="$(arg robot_name)" load_gripper="$(arg load_gripper)"/>
-  </xacro:if>
-  <xacro:unless value="$(arg load_gazebo)">
-    <xacro:panda_arm />
-  </xacro:unless>
+  <xacro:include filename="$(find franka_panda_description)/robots/panda.gazebo.xacro"       />
+  <xacro:include filename="$(find franka_panda_description)/robots/panda.transmission.xacro" />
+  <xacro:panda_arm          arm_id="$(arg robot_name)" in_gazebo="true" xyz="0 0 0" rpy="0 0 0" />
+  <xacro:panda_gazebo       robot_name="$(arg robot_name)" load_gripper="$(arg load_gripper)"/>
+  <xacro:panda_transmission robot_name="$(arg robot_name)" load_gripper="$(arg load_gripper)"/>
   <!-- Default Panda Gripper -->
   <xacro:if value="$(arg load_gripper)">

Commit message: chore: minor changes

File: robots/panda_arm.xacro (robot description, xacro)
@@ -1,6 +1,5 @@
 <?xml version='1.0'?>
 <robot xmlns:xacro="http://www.ros.org/wiki/xacro" name="panda">
-  <xacro:macro name="panda_arm" params="arm_id:='panda' description_pkg:='franka_panda_description'
-				connected_to:='' in_gazebo='false' xyz:='0 0 0' rpy:='0 0 0'">
+  <xacro:macro name="panda_arm" params="arm_id:='panda' description_pkg:='franka_panda_description' connected_to:='' in_gazebo='false' xyz:='0 0 0' rpy:='0 0 0'">
     <xacro:property name="joint_damping" value="1.0"/>
     <xacro:unless value="${not connected_to}">
@@ -149,9 +148,9 @@
         </geometry>
       </visual>
-      <collision>
+      <!-- <collision>
         <geometry>
           <mesh filename="package://${description_pkg}/meshes/collision/link5.stl"/>
         </geometry>
-      </collision>
+      </collision> -->
       <inertial>
         <origin xyz="-1.1953e-02 4.1065e-02 -3.8437e-02" rpy="0 0 0"/>
@@ -175,9 +174,9 @@
         </geometry>
       </visual>
-      <collision>
+      <!-- <collision>
         <geometry>
           <mesh filename="package://${description_pkg}/meshes/collision/link6.stl"/>
         </geometry>
-      </collision>
+      </collision> -->
       <inertial>
         <origin xyz="6.0149e-02 -1.4117e-02 -1.0517e-02" rpy="0 0 0"/>
@@ -201,9 +200,9 @@
         </geometry>
       </visual>
-      <collision>
+      <!-- <collision>
         <geometry>
           <mesh filename="package://${description_pkg}/meshes/collision/link7.stl"/>
         </geometry>
-      </collision>
+      </collision> -->
       <inertial>
         <origin xyz="1.0517e-02 -4.252e-03 6.1597e-02" rpy="0 0 0"/>

File: urdf/camera/_d415.gazebo.xacro (robot description, xacro)
@@ -6,5 +6,5 @@
 -->
 <robot xmlns:xacro="http://ros.org/wiki/xacro">
-  <xacro:macro name="gazebo_d415" params="camera_name reference_link topics_ns depth_optical_frame color_optical_frame infrared1_optical_frame infrared2_optical_frame" >
+  <xacro:macro name="gazebo_d415" params="camera_name reference_link topics_ns depth_optical_frame color_optical_frame infrared1_optical_frame infrared2_optical_frame">
     <!-- Load parameters to model's main link-->
     <xacro:property name="deg_to_rad" value="0.01745329251994329577" />
@@ -45,5 +45,5 @@
         <always_on>1</always_on>
         <update_rate>15</update_rate>
-        <visualize>1</visualize>
+        <visualize>0</visualize>
       </sensor>
       <sensor name="${camera_name}ired1" type="camera">
@@ -116,24 +116,24 @@
       <plugin name="${topics_ns}" filename="librealsense_gazebo_plugin.so">
         <prefix>${camera_name}</prefix>
-      	<depthUpdateRate>10.0</depthUpdateRate>
-      	<colorUpdateRate>10.0</colorUpdateRate>
-      	<!-- <infraredUpdateRate>10.0</infraredUpdateRate> -->
-      	<depthTopicName>depth/image_raw</depthTopicName>
-      	<depthCameraInfoTopicName>depth/camera_info</depthCameraInfoTopicName>
-      	<colorTopicName>color/image_raw</colorTopicName>
-      	<colorCameraInfoTopicName>color/camera_info</colorCameraInfoTopicName>
-      	<!--<infrared1TopicName>infra1/image_raw</infrared1TopicName>
+        <depthUpdateRate>10.0</depthUpdateRate>
+        <colorUpdateRate>10.0</colorUpdateRate>
+        <!-- <infraredUpdateRate>10.0</infraredUpdateRate> -->
+        <depthTopicName>depth/image_raw</depthTopicName>
+        <depthCameraInfoTopicName>depth/camera_info</depthCameraInfoTopicName>
+        <colorTopicName>color/image_raw</colorTopicName>
+        <colorCameraInfoTopicName>color/camera_info</colorCameraInfoTopicName>
+        <!--<infrared1TopicName>infra1/image_raw</infrared1TopicName>
       	<infrared1CameraInfoTopicName>infra1/camera_info</infrared1CameraInfoTopicName>
       	<infrared2TopicName>infra2/image_raw</infrared2TopicName>
       	<infrared2CameraInfoTopicName>infra2/camera_info</infrared2CameraInfoTopicName> -->
-      	<colorOpticalframeName>${color_optical_frame}</colorOpticalframeName>
-      	<depthOpticalframeName>${depth_optical_frame}</depthOpticalframeName>
-      	<infrared1OpticalframeName>${infrared1_optical_frame}</infrared1OpticalframeName>
-      	<infrared2OpticalframeName>${infrared2_optical_frame}</infrared2OpticalframeName>
-      	<rangeMinDepth>0.45</rangeMinDepth>
-      	<rangeMaxDepth>10.0</rangeMaxDepth>
-      	<pointCloud>true</pointCloud>
-      	<pointCloudTopicName>depth/points</pointCloudTopicName>
-      	<pointCloudCutoff>0.45</pointCloudCutoff>
+        <colorOpticalframeName>${color_optical_frame}</colorOpticalframeName>
+        <depthOpticalframeName>${depth_optical_frame}</depthOpticalframeName>
+        <infrared1OpticalframeName>${infrared1_optical_frame}</infrared1OpticalframeName>
+        <infrared2OpticalframeName>${infrared2_optical_frame}</infrared2OpticalframeName>
+        <rangeMinDepth>0.45</rangeMinDepth>
+        <rangeMaxDepth>10.0</rangeMaxDepth>
+        <pointCloud>true</pointCloud>
+        <pointCloudTopicName>depth/points</pointCloudTopicName>
+        <pointCloudCutoff>0.45</pointCloudCutoff>
         <pointCloudCutoffMax>1.5</pointCloudCutoffMax>
       </plugin>

File: urdf/camera/_d415.urdf.xacro (robot description, xacro)
@@ -6,5 +6,6 @@
 aluminum peripherial evaluation case.
 -->
-<robot name="sensor_d415" xmlns:xacro="http://ros.org/wiki/xacro">
+<robot name="sensor_d415"
+  xmlns:xacro="http://ros.org/wiki/xacro">
   <!-- Includes -->
   <xacro:include filename="$(find franka_panda_description)/urdf/camera/_d415.gazebo.xacro"/>
@@ -29,5 +30,5 @@
     <xacro:property name="d415_cam_depth_pz" value="${d415_cam_height/2}"/>
     <material name="${name}_aluminum">
-	  <color rgba="0.5 0.5 0.5 1"/>
+      <color rgba="0.5 0.5 0.5 1"/>
     </material>
     <!-- camera body, with origin at bottom screw mount -->
@@ -45,7 +46,7 @@
     <link name="${name}_link">
       <visual>
-      <origin xyz="${d415_cam_mount_from_center_offset} ${-d415_cam_depth_py} 0" rpy="${M_PI/2} 0 ${M_PI/2}"/>
+        <origin xyz="${d415_cam_mount_from_center_offset} ${-d415_cam_depth_py} 0" rpy="${M_PI/2} 0 ${M_PI/2}"/>
         <geometry>
-	         <mesh filename="package://franka_panda_description/meshes/camera/d415.stl" />
+          <mesh filename="package://franka_panda_description/meshes/camera/d415.stl" />
         </geometry>
         <material name="${name}_aluminum"/>
@@ -66,55 +67,55 @@
     <!-- camera depth joints and links -->
     <joint name="${name}_depth_joint" type="fixed">
-    <origin xyz="0 0 0" rpy="0 0 0"/>
-    <parent link="${name}_link"/>
-    <child link="${name}_depth_frame" />
+      <origin xyz="0 0 0" rpy="0 0 0"/>
+      <parent link="${name}_link"/>
+      <child link="${name}_depth_frame" />
     </joint>
     <link name="${name}_depth_frame"/>
     <joint name="${name}_depth_optical_joint" type="fixed">
-    <origin xyz="0 0 0" rpy="${-M_PI/2} 0 ${-M_PI/2}" />
-    <parent link="${name}_depth_frame" />
-    <child link="${name}_depth_optical_frame" />
+      <origin xyz="0 0 0" rpy="${-M_PI/2} 0 ${-M_PI/2}" />
+      <parent link="${name}_depth_frame" />
+      <child link="${name}_depth_optical_frame" />
     </joint>
     <link name="${name}_depth_optical_frame"/>
     <!-- camera left IR joints and links -->
     <joint name="${name}_left_ir_joint" type="fixed">
-    <origin xyz="0 ${d415_cam_depth_to_left_ir_offset} 0" rpy="0 0 0" />
-    <!-- <parent link="${name}_link" /> -->
-    <parent link="${name}_depth_frame" />
-    <child link="${name}_left_ir_frame" />
+      <origin xyz="0 ${d415_cam_depth_to_left_ir_offset} 0" rpy="0 0 0" />
+      <!-- <parent link="${name}_link" /> -->
+      <parent link="${name}_depth_frame" />
+      <child link="${name}_left_ir_frame" />
     </joint>
     <link name="${name}_left_ir_frame"/>
     <joint name="${name}_left_ir_optical_joint" type="fixed">
-    <origin xyz="0 0 0" rpy="${-M_PI/2} 0 ${-M_PI/2}" />
-    <parent link="${name}_left_ir_frame" />
-    <child link="${name}_left_ir_optical_frame" />
+      <origin xyz="0 0 0" rpy="${-M_PI/2} 0 ${-M_PI/2}" />
+      <parent link="${name}_left_ir_frame" />
+      <child link="${name}_left_ir_optical_frame" />
     </joint>
     <link name="${name}_left_ir_optical_frame"/>
     <!-- camera right IR joints and links -->
     <joint name="${name}_right_ir_joint" type="fixed">
-    <origin xyz="0 ${d415_cam_depth_to_right_ir_offset} 0" rpy="0 0 0" />
-    <!-- <parent link="${name}_link" /> -->
-    <parent link="${name}_depth_frame" />
-    <child link="${name}_right_ir_frame" />
+      <origin xyz="0 ${d415_cam_depth_to_right_ir_offset} 0" rpy="0 0 0" />
+      <!-- <parent link="${name}_link" /> -->
+      <parent link="${name}_depth_frame" />
+      <child link="${name}_right_ir_frame" />
     </joint>
     <link name="${name}_right_ir_frame"/>
     <joint name="${name}_right_ir_optical_joint" type="fixed">
-    <origin xyz="0 0 0" rpy="${-M_PI/2} 0 ${-M_PI/2}" />
-    <parent link="${name}_right_ir_frame" />
-    <child link="${name}_right_ir_optical_frame" />
+      <origin xyz="0 0 0" rpy="${-M_PI/2} 0 ${-M_PI/2}" />
+      <parent link="${name}_right_ir_frame" />
+      <child link="${name}_right_ir_optical_frame" />
     </joint>
     <link name="${name}_right_ir_optical_frame"/>
     <!-- camera color joints and links -->
     <joint name="${name}_color_joint" type="fixed">
-        <origin xyz="0 ${d415_cam_depth_to_color_offset} 0" rpy="0 0 0" />
-        <!-- <parent link="${name}_link" /> -->
-        <parent link="${name}_depth_frame" />
-        <child link="${name}_color_frame" />
+      <origin xyz="0 ${d415_cam_depth_to_color_offset} 0" rpy="0 0 0" />
+      <!-- <parent link="${name}_link" /> -->
+      <parent link="${name}_depth_frame" />
+      <child link="${name}_color_frame" />
     </joint>
     <link name="${name}_color_frame"/>
     <joint name="${name}_color_optical_joint" type="fixed">
-    <origin xyz="0 0 0" rpy="${-M_PI/2} 0 ${-M_PI/2}" />
-    <parent link="${name}_color_frame" />
-    <child link="${name}_color_optical_frame" />
+      <origin xyz="0 0 0" rpy="${-M_PI/2} 0 ${-M_PI/2}" />
+      <parent link="${name}_color_frame" />
+      <child link="${name}_color_optical_frame" />
     </joint>
     <link name="${name}_color_optical_frame"/>

Commit message: feat: remove link 567 collision from franka

File: robots/panda_arm.xacro (robot description, xacro)
@@ -149,9 +149,9 @@
         </geometry>
       </visual>
-      <collision>
+      <!-- <collision>
         <geometry>
           <mesh filename="package://${description_pkg}/meshes/collision/link5.stl"/>
         </geometry>
-      </collision>
+      </collision> -->
       <inertial>
         <origin xyz="-1.1953e-02 4.1065e-02 -3.8437e-02" rpy="0 0 0"/>
@@ -175,9 +175,9 @@
         </geometry>
       </visual>
-      <collision>
+      <!-- <collision>
         <geometry>
           <mesh filename="package://${description_pkg}/meshes/collision/link6.stl"/>
         </geometry>
-      </collision>
+      </collision> -->
       <inertial>
         <origin xyz="6.0149e-02 -1.4117e-02 -1.0517e-02" rpy="0 0 0"/>
@@ -201,9 +201,9 @@
         </geometry>
       </visual>
-      <collision>
+      <!-- <collision>
         <geometry>
           <mesh filename="package://${description_pkg}/meshes/collision/link7.stl"/>
         </geometry>
-      </collision>
+      </collision> -->
       <inertial>
         <origin xyz="1.0517e-02 -4.252e-03 6.1597e-02" rpy="0 0 0"/>
