Commit message: perf (d435): deactivate collision and inertia

File: urdf/camera/_d435.urdf.xacro (robot description, xacro)
@@ -53,16 +53,16 @@
         <material name="${name}_aluminum"/>
       </visual>
-      <collision>
+      <!-- <collision>
         <origin xyz="0 ${-d435_cam_depth_py} 0" rpy="0 0 0"/>
         <geometry>
         <box size="${d435_cam_depth} ${d435_cam_width} ${d435_cam_height}"/>
         </geometry>
-      </collision>
-      <inertial>
-        <!-- The following are not reliable values, and should not be used for modeling -->
+      </collision> -->
+      <!-- The following are not reliable values, and should not be used for modeling -->
+      <!-- <inertial>
         <mass value="0.564" />
         <origin xyz="0 0 0" />
         <inertia ixx="0.003881243" ixy="0.0" ixz="0.0" iyy="0.000498940" iyz="0.0" izz="0.003879257" />
-      </inertial>
+      </inertial> -->
     </link>
     <!-- camera depth joints and links -->

Commit message: style: clean up file

File: urdf/camera/_d435.urdf.xacro (robot description, xacro)
@@ -47,7 +47,5 @@
       <origin xyz="${d435_cam_mount_from_center_offset} ${-d435_cam_depth_py} 0" rpy="${M_PI/2} 0 ${M_PI/2}"/>
         <geometry>
-          <!-- <box size="${d435_cam_width} ${d435_cam_height} ${d435_cam_depth}"/> -->
           <mesh filename="package://franka_panda_description/meshes/camera/d435.dae" />
-          <!--<mesh filename="package://realsense2_description/meshes/d435/d435.dae" />-->
         </geometry>
         <material name="${name}_aluminum"/>
